File: PCB/PiicoDev-Accelerometer-LIS3DH.kicad_sch (KiCad schematic)
At the start: 23 parts, among them J1 , J2 , J3 Conn_PiicoDev_header_01x04_Ma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, J4 INT, SW1 ASW, U1 LIS3DH

Commit message: add documents and link CAD
Parts:
- added R5: 120R, Resistor_SMD:R_0402_1005Metric, symbol Device:R
Connections:
- net SDA: now also R5.1; no longer U1.6 (SDA/SDI/SDO)
- new net: R5.2, U1.6 (SDA/SDI/SDO)
Other:
- note added: "CS Pin pulled high: Device permanently configured for I2C operation R5 120R damps potentially destructive undershoot (for long buses)."
- note removed: "CS Pin pulled high: Device permanently configured for I2C operation"
Changed lines of the file:
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@@
   (title_block
     (title "PiicoDev 3-Axis Accelerometer LIS3DH")
-    (date "2022-06-23")
-    (rev "v00")
+    (date "2022-07-01")
+    (rev "v10")
     (company "Core Electronics")
     (comment 1 "Designed by Michael Ruppe at")
@@
     (stroke (width 0) (type default) (color 0 0 0 0))
   )
-  (wire (pts (xy 173.99 82.55) (xy 181.61 82.55))
+  (wire (pts (xy 152.4 82.55) (xy 181.61 82.55))
     (stroke (width 0) (type default) (color 0 0 0 0))
   )
@@
     (stroke (width 0) (type default) (color 0 0 0 0))
   )
-  (wire (pts (xy 173.99 80.01) (xy 181.61 80.01))
-    (stroke (width 0) (type default) (color 0 0 0 0))
-  )
   (polyline (pts (xy 154.94 182.88) (xy 154.94 196.85))
     (stroke (width 0) (type default) (color 0 0 0 0))
@@
     (stroke (width 0) (type default) (color 0 0 0 0))
   )
+  (wire (pts (xy 161.29 80.01) (xy 181.61 80.01))
+    (stroke (width 0) (type default) (color 0 0 0 0))
+  )
   (polyline (pts (xy 175.26 196.85) (xy 166.37 196.85))
     (stroke (width 0) (type default) (color 0 0 0 0))
@@
   )
   (wire (pts (xy 167.64 38.1) (xy 167.64 39.37))
+    (stroke (width 0) (type default) (color 0 0 0 0))
+  )
+  (wire (pts (xy 152.4 80.01) (xy 153.67 80.01))
     (stroke (width 0) (type default) (color 0 0 0 0))
   )
@@
     (effects (font (size 2.0066 2.0066)) (justify left bottom))
   )
-  (text "CS Pin pulled high:\nDevice permanently configured for I2C operation"
-    (at 142.24 110.49 0)
+  (text "CS Pin pulled high:\nDevice permanently configured for I2C operation\n\nR5 120R damps potentially destructive undershoot (for long buses).\n"
+    (at 139.7 114.3 0)
     (effects (font (size 1.27 1.27)) (justify left bottom))
   )
@@
     (effects (font (size 1.27 1.27)) (justify right bottom))
   )
-  (label "SCL" (at 173.99 82.55 180)
+  (label "SCL" (at 152.4 82.55 180)
     (effects (font (size 1.27 1.27)) (justify right bottom))
   )
@@
     (effects (font (size 1.27 1.27)) (justify left bottom))
   )
-  (label "SDA" (at 173.99 80.01 180)
+  (label "SDA" (at 152.4 80.01 180)
     (effects (font (size 1.27 1.27)) (justify right bottom))
   )
@@
     (pin "2")
   )
+  (symbol (lib_id "Device:R") (at 157.48 80.01 90) (unit 1)
+    (in_bom yes) (on_board yes)
+    (property "Reference" "R5" (id 0) (at 161.29 78.74 90))
+    (property "Value" "120R" (id 1) (at 157.48 80.01 90))
+    (property "Footprint" "Resistor_SMD:R_0402_1005Metric" (id 2) (at 157.48 81.788 90)
+      (effects (font (size 1.27 1.27)) hide)
+    )
+    (property "Datasheet" "~" (id 3) (at 157.48 80.01 0)
+      (effects (font (size 1.27 1.27)) hide)
+    )
+    (pin "1")
+    (pin "2")
+  )
   (symbol (lib_id "Device:C") (at 180.34 43.18 0) (unit 1)
     (in_bom yes) (on_board yes) (fields_autoplaced)
@@
       (reference "R4") (unit 1) (value "10k") (footprint "Resistor_SMD:R_0402_1005Metric")
     )
+    (path "/9680e7f9-3777-4a06-8ba8-1a6a4b022a76"
+      (reference "R5") (unit 1) (value "120R") (footprint "Resistor_SMD:R_0402_1005Metric")
+    )
     (path "/4221e810-476b-456b-986f-2282e69472e1"
